File: PCBTP6_TDII/TP6.kicad_pcb (KiCad board)
At the start: 2 copper layers, 121.9 x 87.6 mm, 30 parts, among them P12 12V, U3.3 NCP1117ST33T3G, U5 LM2575-5.0, X1 12MHz

Commit message: Terminado el pcb
Parts:
- C12, C5, C7, C8, R1, R3, RV1, ULPC1, X1: moved to B.Cu
- moved D1 157.0 mm to (178.9, 222.0), turned to 90 degrees
- moved RV1 155.7 mm to (219.4, 211.7), turned to 180 degrees
- moved PJTAG1 153.8 mm to (231.1, 209.3), turned to 90 degrees
- moved L1 144.7 mm to (184.5, 216.5)
- moved FB2 139.8 mm to (224.0, 224.5)
- moved FB1 137.8 mm to (224.0, 217.5)
- moved U5 133.7 mm to (183.8, 210.3)
- moved U3.3 127.8 mm to (199.0, 222.5), turned to 180 degrees
- moved P12 124.5 mm to (168.8, 215.0), turned to 90 degrees
- moved C11 122.0 mm to (235.0, 221.0), turned to 270 degrees
- moved C10 118.6 mm to (213.5, 221.0), turned to 270 degrees
- moved C2 114.4 mm to (191.0, 221.5), turned to 270 degrees
- moved C1 114.3 mm to (175.3, 215.0), turned to 270 degrees
- moved C3 114.3 mm to (206.5, 221.0), turned to 270 degrees
- moved PDAC1 112.9 mm to (223.3, 198.1), turned to 270 degrees
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Routing:
- net GND: track 0.00 -> 232.1 mm, vias 0 -> 5
- net +3.3V: track 0.00 -> 130.4 mm, vias 0 -> 3
- net GNDA: track 0.00 -> 110.9 mm, vias 0 -> 1
- net N-000003: track 0.00 -> 88.9 mm, vias 0 -> 1
- net N-0000031: track 0.00 -> 48.4 mm, vias 0 -> 2
- net +3.3VADC: track 0.00 -> 48.0 mm, vias 0 -> 1
- net N-0000032: track 0.00 -> 28.6 mm, vias 0 -> 1
- net N-0000028: track 0.00 -> 28.5 mm, vias 0 -> 1
- net N-0000034: track 0.00 -> 26.8 mm, vias 0 -> 1
- net +5V: track 0.00 -> 18.4 mm
- net N-0000089: track 0.00 -> 18.1 mm, vias 0 -> 2
- net N-0000088: track 0.00 -> 15.6 mm, vias 0 -> 2
- net N-0000086: track 0.00 -> 13.0 mm
- net N-0000092: track 0.00 -> 10.00 mm
- net N-0000087: track 0.00 -> 9.36 mm
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- added copper zone on B.Cu, net GND
- added copper zone on F.Cu, net GND
Other:
- board size 121.9 x 87.6 mm -> 83 x 41.5 mm
- net class Default: clearance 0.254 -> 0.1
- net class Micro added: clearance 0.1, trace_width 0.508, via_dia 0.889, via_drill 0.635
- rule trace_clearance: 0.254 -> 0.1
